Commit message: made all the requirements to control robot in gazebo

File: src/my_robot_description/urdf/turret.urdf.xacro (robot description, xacro)
@@ -3,29 +3,102 @@
 	<link name="base_link">
 		<visual>
+			<origin xyz='0.000009 -0.000032 3.1399' rpy='0 0 0'/>
 			<geometry>
 				<mesh filename="package://my_robot_description/meshes/bottombase.stl"/>
 			</geometry>
 		</visual>
+		<inertial>
+  			<mass value="1.0"/>
+  			<origin xyz="0 0 0"/>
+  			<inertia
+    			ixx="0.1" ixy="0" ixz="0"
+    			iyy="0.1" iyz="0"
+    			izz="0.1"/>
+		</inertial>
 	</link>
 	<link name="base_top">
 		<visual>
+			<origin xyz='0 0 0' rpy='0 0 0'/>
 			<geometry>
 				<mesh filename="package://my_robot_description/meshes/basetop.stl"/>
 			</geometry>
 		</visual>
+		<inertial>
+  			<mass value="1.0"/>
+  			<origin xyz="0 0 0"/>
+  			<inertia
+    			ixx="0.1" ixy="0" ixz="0"
+    			iyy="0.1" iyz="0"
+    			izz="0.1"/>
+		</inertial>
 	</link>
+	<joint name='base_to_top' type='fixed'>
+		<parent link='base_link'/>
+		<child link='base_top'/>
+		<origin xyz='0.63776 0.019067 5.0907' rpy='0 0 0.20868902'/>
+	</joint>
 	<link name="rotating_support">
 		<visual>
+			<origin xyz='0.096907 0.65344 7.582' rpy='0 0 0'/>
 			<geometry>
-				<mesh filename="package://my_robot_description/meshes/rotatingbase.stl"/>
+				<mesh filename="package://my_robot_description/meshes/rotatingsupport.stl"/>
 			</geometry>
 		</visual>
+		<inertial>
+  			<mass value="1.0"/>
+  			<origin xyz="0 0 0"/>
+  			<inertia
+    			ixx="0.1" ixy="0" ixz="0"
+    			iyy="0.1" iyz="0"
+    			izz="0.1"/>
+		</inertial>
 	</link>
 	<link name="barrel">
-                <visual>
-                        <geometry>
-                                <mesh filename="package://my_robot_description/meshes/barrel.stl"/>
-                        </geometry>
-                </visual>
-        </link>
+        <visual>
+			<origin xyz='-0.43407 0.027148 12.121' rpy='0 0 3.141592654'/>
+            <geometry>
+                <mesh filename="package://my_robot_description/meshes/barrel.stl"/>
+            </geometry>
+        </visual>
+		<inertial>
+  			<mass value="1.0"/>
+  			<origin xyz="0 0 0"/>
+  			<inertia
+    			ixx="0.1" ixy="0" ixz="0"
+    			iyy="0.1" iyz="0"
+    			izz="0.1"/>
+		</inertial>
+    </link>
+	<joint name='joint1' type='revolute'>
+		<parent link='base_top'/>
+		<child link='rotating_support'/>
+		<origin xyz='1.04 -0.03729 5.506'/>
+		<axis xyz='0 0 1'/>
+		<limit lower='-1.5708' upper='1.5708' effort='10' velocity='1'/>
+	</joint>
+	<joint name='joint2' type='revolute'>
+		<parent link='rotating_support'/>
+		<child link='barrel'/>
+		<origin xyz='7.94 -0.06256 11.21'/>
+		<axis xyz='1 0 0'/>
+		<limit lower='-1.5708' upper='1.5708' effort='10' velocity='1'/>
+	</joint>
+	<ros2_control name='GazeboSystem' type='system'>
+		<hardware>
+			<plugin>gz_ros2_control/GazeboSimSystem</plugin>
+		</hardware>
+		<joint name='joint1'>
+			<command_interface name='position'/>
+			<state_interface name='position'/>
+			<state_interface name='velocity'/>
+		</joint>
+		<joint name='joint2'>
+			<command_interface name='position'/>
+			<state_interface name='position'/>
+			<state_interface name='velocity'/>
+		</joint>
+	</ros2_control>
+	<gazebo reference="base_link">
+  		<static>true</static>
+	</gazebo>
 </robot>

Commit message: made some changes asper tutorial

File: src/my_robot_description/urdf/turret.urdf.xacro (robot description, xacro)
@@ -1,11 +1,17 @@
 <?xml version="1.0"?>
-<robot name="turret">
+<robot xmlns:xacro="http://www.ros.org/wiki/xacro" name="turret">
 	<link name="base_link">
 		<visual>
-			<origin xyz='0.000009 -0.000032 3.1399' rpy='0 0 0'/>
+			<origin xyz='-1.02426 0.023517 -0.004124' rpy='0 0 0'/>
 			<geometry>
 				<mesh filename="package://my_robot_description/meshes/bottombase.stl"/>
 			</geometry>
 		</visual>
+		<collision>
+			<origin xyz='-1.02426 0.023517 -0.004124' rpy='0 0 0'/>
+			<geometry>
+				<mesh filename="package://my_robot_description/meshes/bottombase.stl"/>
+			</geometry>
+		</collision>
 		<inertial>
   			<mass value="1.0"/>
@@ -19,9 +25,15 @@
 	<link name="base_top">
 		<visual>
-			<origin xyz='0 0 0' rpy='0 0 0'/>
+			<origin xyz='-0.379516 0.107647 5.09452' rpy='0 0 0.2'/>
 			<geometry>
 				<mesh filename="package://my_robot_description/meshes/basetop.stl"/>
 			</geometry>
 		</visual>
+		<collision>
+			<origin xyz='-0.379516 0.107647 5.09452' rpy='0 0 0.2'/>
+			<geometry>
+				<mesh filename="package://my_robot_description/meshes/basetop.stl"/>
+			</geometry>
+		</collision>
 		<inertial>
   			<mass value="1.0"/>
@@ -36,13 +48,19 @@
 		<parent link='base_link'/>
 		<child link='base_top'/>
-		<origin xyz='0.63776 0.019067 5.0907' rpy='0 0 0.20868902'/>
+		<origin xyz='0 0 0' rpy='0 0 0'/>
 	</joint>
 	<link name="rotating_support">
 		<visual>
-			<origin xyz='0.096907 0.65344 7.582' rpy='0 0 0'/>
+			<origin xyz='0 0 0' rpy='0 0 0'/>
 			<geometry>
 				<mesh filename="package://my_robot_description/meshes/rotatingsupport.stl"/>
 			</geometry>
 		</visual>
+		<collision>
+			<origin xyz='0 0 0' rpy='0 0 0'/>
+			<geometry>
+				<mesh filename="package://my_robot_description/meshes/rotatingsupport.stl"/>
+			</geometry>
+		</collision>
 		<inertial>
   			<mass value="1.0"/>
@@ -56,9 +74,15 @@
 	<link name="barrel">
         <visual>
-			<origin xyz='-0.43407 0.027148 12.121' rpy='0 0 3.141592654'/>
+			<origin xyz='0 0 0' rpy='0 0 0'/>
             <geometry>
                 <mesh filename="package://my_robot_description/meshes/barrel.stl"/>
             </geometry>
         </visual>
+		<collision>
+			<origin xyz='0 0 0' rpy='0 0 0'/>
+            <geometry>
+                <mesh filename="package://my_robot_description/meshes/barrel.stl"/>
+            </geometry>
+        </collision>
 		<inertial>
   			<mass value="1.0"/>
@@ -73,5 +97,5 @@
 		<parent link='base_top'/>
 		<child link='rotating_support'/>
-		<origin xyz='1.04 -0.03729 5.506'/>
+		<origin xyz='0.021961 0.047853 5.74467'/>
 		<axis xyz='0 0 1'/>
 		<limit lower='-1.5708' upper='1.5708' effort='10' velocity='1'/>
@@ -80,5 +104,5 @@
 		<parent link='rotating_support'/>
 		<child link='barrel'/>
-		<origin xyz='7.94 -0.06256 11.21'/>
+		<origin xyz='6.9 -0.025264 5.69999'/>
 		<axis xyz='1 0 0'/>
 		<limit lower='-1.5708' upper='1.5708' effort='10' velocity='1'/>
@@ -102,3 +126,8 @@
   		<static>true</static>
 	</gazebo>
+	<gazebo>
+  		<plugin filename="libgz_ros2_control-system.so"
+        	name="gz_ros2_control::GazeboSimROS2ControlPlugin">
+		</plugin>
+	</gazebo>
 </robot>
